Commit message: update URDF and SRDF for 1DOF model

File: ModularBot/urdf/ModularBot.urdf (robot description, URDF)
Before this commit: robot ModularBot, 10 links, 9 joints
Links:
- removed link L_0_A
Joints:
- removed joint L_0_A_fixed_joint_0
- joint fixed_J1_A: origin xyz=0.0 0.0 0.06 rpy=0.0 -0.0 0.0 -> xyz=0.0 0.0 0.0 rpy=0.0 -0.0 0.0; parent L_0_A -> base_link

Commit message: cleanup and rename ModularBot ->ModularBot_1DOF

File: ModularBot/urdf/ModularBot.urdf (robot description, URDF)
Before this commit: robot ModularBot, 9 links, 8 joints
Links:
- link J1_A_stator: geometry collision mesh filename=package://ModularBot_1DOF/database/modular/meshes/simple/el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 scale=0.001 0.001 0.001; visual mesh filename=package://ModularBot_1DOF/database/modular/meshes/elbow_bas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 scale=0.001 0.001 0.001
- link L_1_A: geometry collision mesh filename=package://ModularBot_1DOF/database/modular/meshes/simple/el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 scale=0.001 0.001 0.001; visual mesh filename=package://ModularBot_1DOF/database/modular/meshes/elbow_lin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 scale=0.001 0.001 0.001
- link base_link: mass 10.0 -> 0.1
- link gripper_A: geometry collision mesh filename=package://ModularBot_1DOF/database/modular/meshes/simple/gr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 scale=0.001 0.001 0.001; visual mesh filename=package://ModularBot_1DOF/database/modular/meshes/gripper_o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 scale=0.001 0.001 0.001
- link gripper_A_leftfinger: geometry collision mesh filename=package://ModularBot_1DOF/database/modular/meshes/simple/fi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 scale=0.001 0.001 0.001; visual mesh filename=package://ModularBot_1DOF/database/modular/meshes/fingerup_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 scale=0.001 0.001 0.001
- link gripper_A_rightfinger: geometry collision mesh filename=package://ModularBot_1DOF/database/modular/meshes/simple/fi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 scale=0.001 0.001 0.001; visual mesh filename=package://ModularBot_1DOF/database/modular/meshes/fingerup_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 scale=0.001 0.001 0.001
