Commit message: add ModularBot_4DOF

File: ModularBot_4DOF/urdf/ModularBot.urdf (robot description, URDF)
Before this commit: robot ModularBot_6DOF, 22 links, 21 joints
Links:
- removed link J5_A_stator
- removed link J6_A_stator
- removed link L_5_A
- removed link L_5_A_rotor_fast
- removed link L_6_A
- removed link L_6_A_rotor_fast
- removed link pen_A
- removed link tool_exchanger_A
- added link TCP_gripper_A
- added link gripper_A, mass 1.182; collision mesh filename=package://ModularBot_4DOF/database/modular/meshes/simple/gr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 scale=0.001 0.001 0.001; visual mesh filename=package://ModularBot_4DOF/database/modular/meshes/gripper_o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 scale=0.001 0.001 0.001
- added link gripper_A_leftfinger, mass 0.001; collision mesh filename=package://ModularBot_4DOF/database/modular/meshes/simple/fi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 scale=0.001 0.001 0.001; visual mesh filename=package://ModularBot_4DOF/database/modular/meshes/fingerup_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 scale=0.001 0.001 0.001
- added link gripper_A_rightfinger, mass 0.001; collision mesh filename=package://ModularBot_4DOF/database/modular/meshes/simple/fi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 scale=0.001 0.001 0.001; visual mesh filename=package://ModularBot_4DOF/database/modular/meshes/fingerup_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 scale=0.001 0.001 0.001
- link J1_A_stator: geometry collision mesh filename=package://ModularBot_4DOF/database/modular/meshes/simple/ya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 scale=0.001 0.001 0.001; visual mesh filename=package://ModularBot_4DOF/database/modular/meshes/yaw_base.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 scale=0.001 0.001 0.001
- link J2_A_stator: geometry collision mesh filename=package://ModularBot_4DOF/database/modular/meshes/simple/el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 scale=0.001 0.001 0.001; visual mesh filename=package://ModularBot_4DOF/database/modular/meshes/elbow_bas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 scale=0.001 0.001 0.001
- link J3_A_stator: mass 2.0554934 -> 1.8627994; geometry collision mesh filename=package://ModularBot_4DOF/database/modular/meshes/simple/el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 scale=0.001 0.001 0.001; visual mesh filename=package://ModularBot_4DOF/database/modular/meshes/elbow_bas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 scale=0.001 0.001 0.001
- link J4_A_stator: geometry collision mesh filename=package://ModularBot_4DOF/database/modular/meshes/simple/el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 scale=0.001 0.001 0.001; visual mesh filename=package://ModularBot_4DOF/database/modular/meshes/elbow_bas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 scale=0.001 0.001 0.001
- link L_1_A: geometry collision mesh filename=package://ModularBot_4DOF/database/modular/meshes/simple/ya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 scale=0.001 0.001 0.001; visual mesh filename=package://ModularBot_4DOF/database/modular/meshes/yaw_link.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 scale=0.001 0.001 0.001
- link L_2_A: geometry collision mesh filename=package://ModularBot_4DOF/database/modular/meshes/simple/el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 scale=0.001 0.001 0.001; visual mesh filename=package://ModularBot_4DOF/database/modular/meshes/elbow_lin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 scale=0.001 0.001 0.001
- link L_3_A: mass 0.42322395 -> 1.1036463; geometry collision mesh filename=package://ModularBot_4DOF/database/modular/meshes/simple/el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 scale=0.001 0.001 0.001; visual mesh filename=package://ModularBot_4DOF/database/modular/meshes/elbow_lin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 scale=0.001 0.001 0.001
- link L_4_A: geometry collision mesh filename=package://ModularBot_4DOF/database/modular/meshes/simple/el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 scale=0.001 0.001 0.001; visual mesh filename=package://ModularBot_4DOF/database/modular/meshes/elbow_lin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 scale=0.001 0.001 0.001
Joints:
- removed joint J5_A
- removed joint J6_A
- removed joint fixed_J5_A
- removed joint fixed_J6_A
- removed joint fixed_L_5_A_rotor_fast
- removed joint fixed_L_6_A_rotor_fast
- removed joint fixed_pen_A
- removed joint tool_exchanger_A_fixed_joint
- added joint fixed_TCP_gripper_A: type fixed, parent gripper_A, child TCP_gripper_A, origin xyz=0.0 0.0 0.1985 rpy=0.0 0.0 0.0, axis 0 0 1
- added joint gripper_A_finger_joint1: type fixed, parent gripper_A, child gripper_A_leftfinger, origin xyz=0 0 0.1275 rpy=0 0 0, axis 0 -1 0, limit lower=0.0 upper=0.05 effort=20.0 velocity=0.2
- added joint gripper_A_finger_joint2: type fixed, parent gripper_A, child gripper_A_rightfinger, origin xyz=0 0 0.1275 rpy=0 0 0, axis 0 1 0, limit lower=0.0 upper=0.05 effort=20.0 velocity=0.2
- added joint gripper_A_fixed_joint: type fixed, parent L_4_A, child gripper_A, origin xyz=0.0 -0.131999958147 -0.0720448848742 rpy=1.57 -0.0 0.0, axis 0 0 1
- joint J3_A: limit lower=-2.8 upper=2.8 effort=147 velocity=3.9 -> lower=-2.0 upper=2.0 effort=147 velocity=3.9; origin xyz=0.0 0.0 0.214 rpy=0.0 -0.0 0.0 -> xyz=0.0 0.0721499771235 0.132057454972 rpy=-1.57 -0.0 0.0
- joint fixed_J4_A: origin xyz=0.0 0.0 0.0 rpy=0.0 -0.0 0.0 -> xyz=0.0 -0.131999958147 -0.0720448848742 rpy=1.57 -0.0 0.0
